File: PCB/miniFPGA/miniFPGA.kicad_pcb (KiCad board)
At the start: 2 copper layers, 24.9 x 57.4 mm, 36 parts, among them J1 USB_B, J2 ICSP_FPGA, U2 MCP2221A-IP, U3 PIC16F13145-IP

Commit message: PCB sources for v3.0
Parts:
- added A1: 8pin proto area, Attila:8pin_proto, F.Cu at (100.4, 173.1)
- added R17: 680Ω, Attila:R_Axial_L3.6mm_D1.6mm_P1.90mm_Vertical, F.Cu at (99.0, 162.6)
- added R18: 4k7, Resistor_THT:R_Axial_DIN0204_L3.6mm_D1.6mm_P5.08mm_Horizontal, F.Cu at (97.4, 128.3)
- added R19: 680Ω, Attila:R_Axial_L3.6mm_D1.6mm_P1.90mm_Vertical, F.Cu at (99.0, 151.0)
- added R20: 680Ω, Attila:R_Axial_L3.6mm_D1.6mm_P1.90mm_Vertical, F.Cu at (99.0, 140.4)
- added R21: 680Ω, Attila:R_Axial_L3.6mm_D1.6mm_P1.90mm_Vertical, F.Cu at (99.0, 130.6)
- added TP1: 1, TestPoint:TestPoint_Pad_1.5x1.5mm, B.Cu at (98.1, 171.7)
- added TP2: 2, TestPoint:TestPoint_Pad_D1.5mm, B.Cu at (100.6, 171.7)
- added TP3: 3, TestPoint:TestPoint_Pad_D1.5mm, B.Cu at (103.2, 171.7)
- added TP4: 4, TestPoint:TestPoint_Pad_D1.5mm, B.Cu at (105.7, 171.7)
- added TP5: 5, TestPoint:TestPoint_Pad_D1.5mm, B.Cu at (105.7, 176.8)
- added TP6: 6, TestPoint:TestPoint_Pad_D1.5mm, B.Cu at (103.2, 176.8)
- added TP7: 7, TestPoint:TestPoint_Pad_D1.5mm, B.Cu at (100.6, 176.8)
- added TP8: 8, TestPoint:TestPoint_Pad_D1.5mm, B.Cu at (98.1, 176.8)
- C1: value 4µ7F -> 4µ7
- J2: value ICSP_FPGA -> ICSP_DEBUG_miniFPGA
- R1, R2, R3, R4: value 10kΩ -> 680Ω; footprint Resistor_THT:R_Axial_DIN0204_L3.6mm_D1.6mm_P5.08mm_Horizontal -> Attila:R_Axial_L3.6mm_D1.6mm_P1.90mm_Vertical
- R11: renamed from R13; value 10kΩ -> 4k7
- R5: renamed from R7; value 10kΩ -> 4k7
- U1: renamed from U2; value MCP2221A-IP -> PIC16F1455-I/P
- moved R13 2.22 mm to (97.1, 126.2), turned to 0 degrees
- moved R12 1.91 mm to (119.3, 126.4), turned to 180 degrees
- moved R5 1.69 mm to (111.1, 129.8)
- moved R1 0.80 mm to (102.8, 130.6)
- moved U1 0.70 mm to (108.3, 133.0)
- moved C1 0.64 mm to (115.5, 129.0)
- moved R2 0.36 mm to (102.8, 140.4)
- moved R3 0.36 mm to (102.8, 151.0)
- moved R4 0.36 mm to (102.8, 162.6)
- moved R10 0.28 mm to (114.9, 151.2)
- moved R7 0.28 mm to (110.9, 151.2)
- moved R8 0.28 mm to (106.9, 151.2)
- moved J1 0.22 mm to (108.2, 120.8)
- moved R9 0.21 mm to (104.9, 152.2)
- renumbered R12 to R10, R14 to R12, R15 to R13, R5 to R14, R6 to R15, R8 to R6, R9 to R7, R10 to R8, R11 to R9, U3 to U2
Connections:
- JP1 pad 2: GNDD -> VDD
- JP2 pad 2: GNDD -> VDD
- JP3 pad 2: GNDD -> VDD
- JP4 pad 2: GNDD -> VDD
- PB1 pad 2: GNDD -> VDD
- PB2 pad 2: GNDD -> VDD
- PB3 pad 2: GNDD -> VDD
- PB4 pad 2: GNDD -> VDD
- R12 pad 1: VDD -> Net-(LED1-A)
- R12 pad 2: Net-(LED1-A) -> VDD
- R13 pad 1: VDD -> Net-(LED2-A)
- R13 pad 2: Net-(LED2-A) -> VDD
Routing:
- net VDD: track 73.8 -> 134.9 mm
- net /URx: track 8.83 -> 27.9 mm
- net Net-(A1-Pin_4): track 0.00 -> 8.87 mm, vias 0 -> 1
- net Net-(A1-Pin_3): track 0.00 -> 7.62 mm, vias 0 -> 1
- net Net-(A1-Pin_8): track 0.00 -> 5.30 mm, vias 0 -> 1
- net Net-(A1-Pin_2): track 0.00 -> 4.30 mm, vias 0 -> 1
- net Net-(A1-Pin_7): track 0.00 -> 3.28 mm, vias 0 -> 1
- net Net-(U1-~{RST}): track 12.1 -> 14.9 mm
- net Net-(A1-Pin_1): track 0.00 -> 2.40 mm, vias 0 -> 1
- net Net-(JP1-A): track 12.0 -> 14.3 mm
- net Net-(JP4-A): track 11.1 -> 13.3 mm
- net Net-(JP3-A): track 12.0 -> 14.3 mm
- net Net-(JP2-A): track 12.0 -> 14.3 mm
- net Net-(A1-Pin_6): track 0.00 -> 1.65 mm, vias 0 -> 1
- net Net-(U1-SDA): track 9.60 -> 8.38 mm
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Other:
- board text added: "PCB Top Side"
- board text added: "PCB bot."
- board text added: "i"
